File: pcb/eagle/esp8255-full-breakout.brd (EAGLE design)
At the start: 23.4 x 35 mm, 12 parts, among them IC1 ESP-12E/F, X1 JST-XH-11-PIN-ROUND-PAD, X2 JST-XH-11-PIN-ROUND-PAD

Commit message: Minor changes
Parts:
- R1, R2, R3, R4, R5: value (none) -> 10KΩ/0805; device adafruit:R1206 -> rcl:R0805
Routing:
- net +3V3: track 64.0 -> 65.4 mm
Other:
- board text added: "R- 10KΩ/0805"
- board text added: "Rev.1.0 (C) 2020"
- board text added: "github.com/CSpyridak is/ESP8266-Breakout"
- board text removed: "10KΩ"
Changed lines of the file:
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@@
 <text x="14.1" y="-0.9" size="0.6096" layer="21">FLASS
 </text>
-<text x="3.1" y="30.1" size="0.8128" layer="22" rot="MR90">10KΩ</text>
-<text x="8.8" y="23.4" size="0.8128" layer="22" rot="MR90">10KΩ</text>
-<text x="13.8" y="23.5" size="0.8128" layer="22" rot="MR90">10KΩ</text>
-<text x="17.2" y="23.5" size="0.8128" layer="22" rot="MR90">10KΩ</text>
-<text x="20.5" y="33.1" size="0.8128" layer="22" rot="MR270">10KΩ</text>
 <text x="16.2" y="34.9" size="0.6096" layer="21" rot="R180">TX</text>
 <text x="13.6" y="34.9" size="0.6096" layer="21" rot="R180">RX</text>
@@
 <text x="22.5" y="5.6" size="0.8128" layer="21" rot="R270">MOSI</text>
 <text x="22.5" y="1.8" size="0.8128" layer="21" rot="R270">10</text>
+<text x="18.9" y="8.3" size="1.4224" layer="26" rot="MR90">R- 10KΩ/0805</text>
+<text x="10.9" y="0.8" size="1.4224" layer="26" rot="MR90">github.com/CSpyridak
+is/ESP8266-Breakout</text>
+<text x="8.4" y="4.1" size="1.4224" layer="26" rot="MR90">Rev.1.0 (C) 2020</text>
 </plain>
 <attributes>
@@
 <attribute name="VALUE" x="19.39" y="36.065" size="1.27" layer="27" rot="R180"/>
 </element>
-<element name="R1" library="adafruit" package="R1206" value="" x="1.81" y="31.87" smashed="yes" rot="MR270">
-<attribute name="VALUE" x="4.223" y="33.267" size="1.27" layer="28" rot="MR270"/>
-</element>
-<element name="R2" library="adafruit" package="R1206" value="" x="21.59" y="31.87" smashed="yes" rot="MR270">
-<attribute name="VALUE" x="24.003" y="33.267" size="1.27" layer="28" rot="MR270"/>
+<element name="R1" library="rcl" library_urn="urn:adsk.eagle:library:334" package="R0805" package3d_urn="urn:adsk.eagle:package:23553/2" value="10KΩ/0805" x="1.81" y="31.87" smashed="yes" rot="MR270">
+<attribute name="POPULARITY" value="86" x="1.81" y="31.87" size="1.778" layer="28" rot="MR270" display="off"/>
+<attribute name="SPICEPREFIX" value="R" x="1.81" y="31.87" size="1.778" layer="28" rot="MR270" display="off"/>
+</element>
+<element name="R2" library="rcl" library_urn="urn:adsk.eagle:library:334" package="R0805" package3d_urn="urn:adsk.eagle:package:23553/2" value="10KΩ/0805" x="21.59" y="31.87" smashed="yes" rot="MR270">
+<attribute name="POPULARITY" value="86" x="21.59" y="31.87" size="1.778" layer="28" rot="MR270" display="off"/>
+<attribute name="SPICEPREFIX" value="R" x="21.59" y="31.87" size="1.778" layer="28" rot="MR270" display="off"/>
 </element>
 <element name="S1" library="switch-tact" package="DTSM-3" value="DTSM-3" x="7.89" y="2.54" smashed="yes"/>
@@
 <element name="X1" library="JST-XH" package="JST-XH-11-PACKAGE-ROUND-PAD" value="JST-XH-11-PIN-ROUND-PAD" x="1.54" y="15.24" smashed="yes" rot="R90"/>
 <element name="X2" library="JST-XH" package="JST-XH-11-PACKAGE-ROUND-PAD" value="JST-XH-11-PIN-ROUND-PAD" x="21.93" y="15.34" smashed="yes" rot="R270"/>
-<element name="R3" library="adafruit" package="R1206" value="" x="12.7" y="24.8" smashed="yes" rot="MR90">
-<attribute name="VALUE" x="10.287" y="23.403" size="1.27" layer="28" rot="MR90"/>
-</element>
-<element name="R4" library="adafruit" package="R1206" value="" x="16.1" y="24.8" smashed="yes" rot="MR270">
-<attribute name="VALUE" x="18.513" y="26.197" size="1.27" layer="28" rot="MR270"/>
-</element>
-<element name="R5" library="adafruit" package="R1206" value="" x="7.7" y="24.9" smashed="yes" rot="MR270">
-<attribute name="VALUE" x="10.113" y="26.297" size="1.27" layer="28" rot="MR270"/>
+<element name="R3" library="rcl" library_urn="urn:adsk.eagle:library:334" package="R0805" package3d_urn="urn:adsk.eagle:package:23553/2" value="10KΩ/0805" x="12.7" y="24.8" smashed="yes" rot="MR90">
+<attribute name="POPULARITY" value="86" x="12.7" y="24.8" size="1.778" layer="28" rot="MR90" display="off"/>
+<attribute name="SPICEPREFIX" value="R" x="12.7" y="24.8" size="1.778" layer="28" rot="MR90" display="off"/>
+</element>
+<element name="R4" library="rcl" library_urn="urn:adsk.eagle:library:334" package="R0805" package3d_urn="urn:adsk.eagle:package:23553/2" value="10KΩ/0805" x="16.1" y="24.8" smashed="yes" rot="MR270">
+<attribute name="POPULARITY" value="86" x="16.1" y="24.8" size="1.778" layer="28" rot="MR270" display="off"/>
+<attribute name="SPICEPREFIX" value="R" x="16.1" y="24.8" size="1.778" layer="28" rot="MR270" display="off"/>
+</element>
+<element name="R5" library="rcl" library_urn="urn:adsk.eagle:library:334" package="R0805" package3d_urn="urn:adsk.eagle:package:23553/2" value="10KΩ/0805" x="7.7" y="24.9" smashed="yes" rot="MR270">
+<attribute name="POPULARITY" value="86" x="7.7" y="24.9" size="1.778" layer="28" rot="MR270" display="off"/>
+<attribute name="SPICEPREFIX" value="R" x="7.7" y="24.9" size="1.778" layer="28" rot="MR270" display="off"/>
 </element>
 <element name="SJ1" library="jumper" library_urn="urn:adsk.eagle:library:252" package="SJ" package3d_urn="urn:adsk.eagle:package:15471/1" value="" x="8" y="29.9" smashed="yes" rot="MR90">
@@
 <wire x1="4.31" y1="25.17" x2="1.54" y2="27.94" width="0.3048" layer="1"/>
 <wire x1="1.54" y1="27.94" x2="1.54" y2="30.178" width="0.3048" layer="16"/>
-<wire x1="1.54" y1="30.178" x2="1.81" y2="30.448" width="0.3048" layer="16"/>
+<wire x1="1.54" y1="30.178" x2="1.81" y2="30.92" width="0.3048" layer="16"/>
 <wire x1="5.19" y1="2.54" x2="3.34" y2="2.54" width="0.3048" layer="1"/>
 <wire x1="3.34" y1="2.54" x2="3.3" y2="2.5" width="0.3048" layer="1"/>
@@
 <wire x1="17.18375" y1="10.3952" x2="15.2" y2="12.37895" width="0.3048" layer="1"/>
 <wire x1="15.2" y1="13.3" x2="15.2" y2="12.37895" width="0.3048" layer="1"/>
-<wire x1="12.7" y1="23.378" x2="12.7" y2="22.678" width="0.3048" layer="16"/>
+<wire x1="12.7" y1="23.85" x2="12.7" y2="22.678" width="0.3048" layer="16"/>
 <wire x1="15.2" y1="20.178" x2="12.7" y2="22.678" width="0.3048" layer="16"/>
 <wire x1="15.2" y1="20.178" x2="15.2" y2="13.3" width="0.3048" layer="16"/>
@@
 <wire x1="18.1" y1="11.3" x2="19.31" y2="11.3" width="0.3048" layer="1"/>
 <contactref element="R4" pad="2"/>
-<wire x1="16.1" y1="23.378" x2="16.4" y2="23.078" width="0.3048" layer="16"/>
+<wire x1="16.1" y1="23.85" x2="16.4" y2="23.078" width="0.3048" layer="16"/>
 <wire x1="16.4" y1="23.078" x2="16.4" y2="13.3" width="0.3048" layer="16"/>
 <via x="16.4" y="13.3" extent="1-16" drill="0.35"/>
@@
 <wire x1="19.9" y1="2.5" x2="18.283" y2="4.117" width="0.3048" layer="16"/>
 <wire x1="18.283" y1="4.117" x2="18.283" y2="12.04305" width="0.3048" layer="16"/>
-<wire x1="21.59" y1="30.448" x2="21.59" y2="29.39" width="0.3048" layer="16"/>
+<wire x1="21.59" y1="30.92" x2="21.59" y2="29.39" width="0.3048" layer="16"/>
 <wire x1="21.59" y1="29.39" x2="19.7" y2="27.5" width="0.3048" layer="16"/>
 <via x="19.7" y="27.5" extent="1-16" drill="0.35"/>
@@
 <wire x1="8.4" y1="19.4" x2="6.3" y2="17.3" width="0.3048" layer="16"/>
 <contactref element="R5" pad="2"/>
-<wire x1="7.7" y1="23.478" x2="8.38" y2="22.798" width="0.3048" layer="16"/>
+<wire x1="7.7" y1="23.95" x2="8.38" y2="22.798" width="0.3048" layer="16"/>
 <wire x1="8.38" y1="22.798" x2="8.38" y2="19.4" width="0.3048" layer="16"/>
 <wire x1="4.27895" y1="17.3" x2="2.7052" y2="18.87375" width="0.3048" layer="1"/>
@@
 <contactref element="R2" pad="1"/>
 <via x="16.5" y="30.6" extent="1-16" drill="0.35"/>
-<wire x1="21.59" y1="33.292" x2="21.5768" y2="33.3052" width="0.3048" layer="16"/>
+<wire x1="21.59" y1="32.82" x2="21.5768" y2="33.3052" width="0.3048" layer="16"/>
 <wire x1="21.5768" y1="33.3052" x2="20.75861875" y2="33.3052" width="0.3048" layer="16"/>
 <wire x1="18.15341875" y1="30.7" x2="16.6" y2="30.7" width="0.3048" layer="16"/>
@@
 <contactref element="R5" pad="1"/>
 <wire x1="10.5" y1="26.4" x2="10.5" y2="16.4" width="0.7" layer="16"/>
-<wire x1="7.7" y1="26.322" x2="7.778" y2="26.4" width="0.3048" layer="16"/>
+<wire x1="7.7" y1="25.85" x2="7.778" y2="26.4" width="0.3048" layer="16"/>
 <wire x1="7.778" y1="26.4" x2="10.4" y2="26.4" width="0.3048" layer="16"/>
 <wire x1="10.4" y1="26.4" x2="10.5" y2="26.4" width="0.3048" layer="16"/>
-<wire x1="16.1" y1="26.222" x2="12.622" y2="29.7" width="0.3048" layer="16"/>
+<wire x1="16.1" y1="25.75" x2="12.622" y2="29.7" width="0.3048" layer="16"/>
 <contactref element="SJ1" pad="1"/>
 <wire x1="16.5" y1="30.6" x2="11.6" y2="30.6" width="0.3048" layer="1"/>
@@
 <wire x1="6.564" y1="29.138" x2="8" y2="29.138" width="0.3048" layer="16"/>
 <wire x1="6.564" y1="29.138" x2="2.41" y2="33.292" width="0.3048" layer="16"/>
-<wire x1="2.41" y1="33.292" x2="1.81" y2="33.292" width="0.3048" layer="16"/>
+<wire x1="2.41" y1="33.292" x2="1.81" y2="32.82" width="0.3048" layer="16"/>
 <wire x1="8" y1="29.138" x2="8" y2="28.8" width="0.8128" layer="16"/>
 <wire x1="10.4" y1="26.4" x2="8" y2="28.8" width="0.8128" layer="16"/>
