File: pcb/eagle/esp8255-full-breakout.sch (EAGLE design)
At the start: 12 parts, among them IC1 ESP-12E/F, X1 JST-XH-11-PIN-ROUND-PAD, X2 JST-XH-11-PIN-ROUND-PAD

Commit message: Minor changes
Parts:
- R1, R2, R3, R4, R5: value (none) -> 10KΩ/0805; device adafruit:R-US_R1206 -> rcl:R-EU_R0805
Changed lines of the file:
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@@
 <part name="GND3" library="supply1" library_urn="urn:adsk.eagle:library:371" deviceset="GND" device=""/>
 <part name="GND4" library="supply1" library_urn="urn:adsk.eagle:library:371" deviceset="GND" device=""/>
-<part name="R1" library="adafruit" deviceset="R-US_" device="R1206"/>
-<part name="R2" library="adafruit" deviceset="R-US_" device="R1206"/>
+<part name="R1" library="rcl" library_urn="urn:adsk.eagle:library:334" deviceset="R-EU_" device="R0805" package3d_urn="urn:adsk.eagle:package:23553/2" value="10KΩ/0805"/>
+<part name="R2" library="rcl" library_urn="urn:adsk.eagle:library:334" deviceset="R-EU_" device="R0805" package3d_urn="urn:adsk.eagle:package:23553/2" value="10KΩ/0805"/>
 <part name="+3V3" library="supply1" library_urn="urn:adsk.eagle:library:371" deviceset="+3V3" device=""/>
 <part name="+3V4" library="supply1" library_urn="urn:adsk.eagle:library:371" deviceset="+3V3" device=""/>
@@
 <part name="FRAME1" library="frames" library_urn="urn:adsk.eagle:library:229" deviceset="A4L-LOC" device=""/>
 <part name="+3V5" library="supply1" library_urn="urn:adsk.eagle:library:371" deviceset="+3V3" device=""/>
-<part name="R3" library="adafruit" deviceset="R-US_" device="R1206"/>
-<part name="R4" library="adafruit" deviceset="R-US_" device="R1206"/>
+<part name="R3" library="rcl" library_urn="urn:adsk.eagle:library:334" deviceset="R-EU_" device="R0805" package3d_urn="urn:adsk.eagle:package:23553/2" value="10KΩ/0805"/>
+<part name="R4" library="rcl" library_urn="urn:adsk.eagle:library:334" deviceset="R-EU_" device="R0805" package3d_urn="urn:adsk.eagle:package:23553/2" value="10KΩ/0805"/>
 <part name="+3V6" library="supply1" library_urn="urn:adsk.eagle:library:371" deviceset="+3V3" device=""/>
 <part name="GND2" library="supply1" library_urn="urn:adsk.eagle:library:371" deviceset="GND" device=""/>
-<part name="R5" library="adafruit" deviceset="R-US_" device="R1206"/>
+<part name="R5" library="rcl" library_urn="urn:adsk.eagle:library:334" deviceset="R-EU_" device="R0805" package3d_urn="urn:adsk.eagle:package:23553/2" value="10KΩ/0805"/>
 <part name="+3V2" library="supply1" library_urn="urn:adsk.eagle:library:371" deviceset="+3V3" device=""/>
 <part name="SJ1" library="jumper" library_urn="urn:adsk.eagle:library:252" deviceset="SJ" device="" package3d_urn="urn:adsk.eagle:package:15471/1"/>
@@
 </instance>
 <instance part="R4" gate="G$1" x="172.72" y="119.38" smashed="yes" rot="R270">
-<attribute name="VALUE" x="169.418" y="123.19" size="1.778" layer="96" rot="R270"/>
+<attribute name="VALUE" x="174.498" y="128.27" size="1.778" layer="96" rot="R270"/>
 </instance>
 <instance part="+3V6" gate="G$1" x="172.72" y="129.54" smashed="yes">
@@
 </instance>
 <instance part="R5" gate="G$1" x="86.36" y="137.16" smashed="yes" rot="R270">
-<attribute name="VALUE" x="83.058" y="140.97" size="1.778" layer="96" rot="R270"/>
+<attribute name="VALUE" x="88.138" y="143.51" size="1.778" layer="96" rot="R270"/>
 </instance>
 <instance part="+3V2" gate="G$1" x="86.36" y="147.32" smashed="yes">
@@
 packages will not be understood (or retained) with this version.
 </note>
+<note version="8.4" severity="warning">
+Since Version 8.4, EAGLE supports properties for SPICE simulation.
+Probes in schematics and SPICE mapping objects found in parts and library devices
+will not be understood with this version. Update EAGLE to the latest version
+for full support of SPICE simulation.
+</note>
 </compatibility>
