File: pcb/eagle/esp8266-breakout.sch (EAGLE design)
At the start: 12 parts, among them IC1 ESP-12E/F, X1 JST-XH-11-PIN-ROUND-PAD, X2 JST-XH-11-PIN-ROUND-PAD

Commit message: V1.1 Done
Other:
- note added: "V1.1"
- moved on the sheet: JP1, R1, R2
Changed lines of the file:
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@@
 <sheet>
 <plain>
+<text x="248.92" y="5.08" size="1.778" layer="94">V1.1</text>
 </plain>
 <instances>
@@
 <attribute name="VALUE" x="109.22" y="157.48" size="2.54" layer="96"/>
 </instance>
-<instance part="JP1" gate="A" x="241.3" y="60.96" smashed="yes">
-<attribute name="NAME" x="234.95" y="71.755" size="1.778" layer="95"/>
-<attribute name="VALUE" x="234.95" y="50.8" size="1.778" layer="96"/>
+<instance part="JP1" gate="A" x="236.22" y="50.8" smashed="yes">
+<attribute name="NAME" x="229.87" y="61.595" size="1.778" layer="95"/>
+<attribute name="VALUE" x="229.87" y="40.64" size="1.778" layer="96"/>
 </instance>
 <instance part="X1" gate="-1" x="33.02" y="111.76" smashed="yes" rot="R180">
@@
 <attribute name="NAME" x="231.14" y="113.538" size="1.524" layer="95"/>
 </instance>
-<instance part="S1" gate="G$1" x="55.88" y="60.96" smashed="yes" rot="R270"/>
-<instance part="S2" gate="G$1" x="55.88" y="35.56" smashed="yes" rot="R270"/>
+<instance part="S1" gate="G$1" x="139.7" y="48.26" smashed="yes" rot="R270"/>
+<instance part="S2" gate="G$1" x="53.34" y="48.26" smashed="yes" rot="R270"/>
 <instance part="+3V1" gate="G$1" x="96.52" y="106.68" smashed="yes">
 <attribute name="VALUE" x="93.98" y="106.68" size="1.778" layer="96" rot="R180"/>
 </instance>
-<instance part="GND1" gate="1" x="223.52" y="53.34" smashed="yes">
-<attribute name="VALUE" x="220.98" y="50.8" size="1.778" layer="96"/>
+<instance part="GND1" gate="1" x="218.44" y="43.18" smashed="yes">
+<attribute name="VALUE" x="215.9" y="40.64" size="1.778" layer="96"/>
 </instance>
 <instance part="GND3" gate="1" x="160.02" y="101.6" smashed="yes">
@@
 <attribute name="VALUE" x="203.2" y="121.92" size="1.778" layer="96"/>
 </instance>
-<instance part="R1" gate="G$1" x="43.18" y="60.96" smashed="yes">
-<attribute name="NAME" x="39.37" y="62.4586" size="1.778" layer="95"/>
-<attribute name="VALUE" x="39.37" y="57.658" size="1.778" layer="96"/>
-</instance>
-<instance part="R2" gate="G$1" x="43.18" y="35.56" smashed="yes">
-<attribute name="NAME" x="39.37" y="37.0586" size="1.778" layer="95"/>
-<attribute name="VALUE" x="39.37" y="32.258" size="1.778" layer="96"/>
-</instance>
-<instance part="+3V3" gate="G$1" x="35.56" y="63.5" smashed="yes">
-<attribute name="VALUE" x="33.02" y="58.42" size="1.778" layer="96" rot="R90"/>
-</instance>
-<instance part="+3V4" gate="G$1" x="35.56" y="38.1" smashed="yes">
-<attribute name="VALUE" x="33.02" y="33.02" size="1.778" layer="96" rot="R90"/>
-</instance>
-<instance part="GND5" gate="1" x="63.5" y="33.02" smashed="yes">
-<attribute name="VALUE" x="60.96" y="30.48" size="1.778" layer="96"/>
-</instance>
-<instance part="GND6" gate="1" x="63.5" y="58.42" smashed="yes">
-<attribute name="VALUE" x="60.96" y="55.88" size="1.778" layer="96"/>
+<instance part="R1" gate="G$1" x="127" y="48.26" smashed="yes">
+<attribute name="NAME" x="123.19" y="49.7586" size="1.778" layer="95"/>
+<attribute name="VALUE" x="123.19" y="44.958" size="1.778" layer="96"/>
+</instance>
+<instance part="R2" gate="G$1" x="40.64" y="48.26" smashed="yes">
+<attribute name="NAME" x="36.83" y="49.7586" size="1.778" layer="95"/>
+<attribute name="VALUE" x="36.83" y="44.958" size="1.778" layer="96"/>
+</instance>
+<instance part="+3V3" gate="G$1" x="119.38" y="50.8" smashed="yes">
+<attribute name="VALUE" x="116.84" y="45.72" size="1.778" layer="96" rot="R90"/>
+</instance>
+<instance part="+3V4" gate="G$1" x="33.02" y="50.8" smashed="yes">
+<attribute name="VALUE" x="30.48" y="45.72" size="1.778" layer="96" rot="R90"/>
+</instance>
+<instance part="GND5" gate="1" x="60.96" y="45.72" smashed="yes">
+<attribute name="VALUE" x="58.42" y="43.18" size="1.778" layer="96"/>
+</instance>
+<instance part="GND6" gate="1" x="147.32" y="45.72" smashed="yes">
+<attribute name="VALUE" x="144.78" y="43.18" size="1.778" layer="96"/>
 </instance>
 <instance part="FRAME1" gate="G$1" x="0" y="0" smashed="yes">
@@
 <attribute name="SHEET" x="230.505" y="5.08" size="2.54" layer="94"/>
 </instance>
-<instance part="+3V5" gate="G$1" x="213.36" y="63.5" smashed="yes">
-<attribute name="VALUE" x="210.82" y="63.5" size="1.778" layer="96" rot="R180"/>
+<instance part="+3V5" gate="G$1" x="208.28" y="53.34" smashed="yes">
+<attribute name="VALUE" x="205.74" y="53.34" size="1.778" layer="96" rot="R180"/>
 </instance>
 <instance part="R3" gate="G$1" x="172.72" y="104.14" smashed="yes" rot="R270">
@@
 <attribute name="VALUE" x="91.44" y="149.86" size="1.778" layer="96" rot="R180"/>
 </instance>
-<instance part="SJ1" gate="1" x="220.98" y="60.96" smashed="yes">
-<attribute name="VALUE" x="218.44" y="57.15" size="1.778" layer="96"/>
+<instance part="SJ1" gate="1" x="215.9" y="50.8" smashed="yes">
+<attribute name="VALUE" x="213.36" y="46.99" size="1.778" layer="96"/>
 </instance>
 <instance part="+3V7" gate="G$1" x="50.8" y="121.92" smashed="yes">
@@
 <pinref part="R1" gate="G$1" pin="2"/>
 <pinref part="S1" gate="G$1" pin="1"/>
-<wire x1="48.26" y1="60.96" x2="50.8" y2="60.96" width="0.1524" layer="91"/>
-<wire x1="50.8" y1="60.96" x2="50.8" y2="68.58" width="0.1524" layer="91"/>
-<wire x1="50.8" y1="68.58" x2="48.26" y2="68.58" width="0.1524" layer="91"/>
-<junction x="50.8" y="60.96"/>
-<label x="48.26" y="68.58" size="1.778" layer="95" rot="R180" xref="yes"/>
+<wire x1="132.08" y1="48.26" x2="134.62" y2="48.26" width="0.1524" layer="91"/>
+<wire x1="134.62" y1="48.26" x2="134.62" y2="55.88" width="0.1524" layer="91"/>
+<wire x1="134.62" y1="55.88" x2="132.08" y2="55.88" width="0.1524" layer="91"/>
+<junction x="134.62" y="48.26"/>
+<label x="132.08" y="55.88" size="1.778" layer="95" rot="R180" xref="yes"/>
 </segment>
 </net>
@@
 <pinref part="R2" gate="G$1" pin="2"/>
 <pinref part="S2" gate="G$1" pin="1"/>
-<wire x1="48.26" y1="35.56" x2="50.8" y2="35.56" width="0.1524" layer="91"/>
-<wire x1="50.8" y1="35.56" x2="50.8" y2="43.18" width="0.1524" layer="91"/>
-<wire x1="50.8" y1="43.18" x2="48.26" y2="43.18" width="0.1524" layer="91"/>
-<junction x="50.8" y="35.56"/>
-<label x="48.26" y="43.18" size="1.778" layer="95" rot="R180" xref="yes"/>
+<wire x1="45.72" y1="48.26" x2="48.26" y2="48.26" width="0.1524" layer="91"/>
+<wire x1="48.26" y1="48.26" x2="48.26" y2="55.88" width="0.1524" layer="91"/>
+<wire x1="48.26" y1="55.88" x2="45.72" y2="55.88" width="0.1524" layer="91"/>
+<junction x="48.26" y="48.26"/>
+<label x="45.72" y="55.88" size="1.778" layer="95" rot="R180" xref="yes"/>
 </segment>
 </net>
@@
 <segment>
 <pinref part="JP1" gate="A" pin="3"/>
-<label x="233.68" y="63.5" size="1.778" layer="95" rot="R180" xref="yes"/>
-<wire x1="238.76" y1="63.5" x2="233.68" y2="63.5" width="0.1524" layer="91"/>
+<label x="228.6" y="53.34" size="1.778" layer="95" rot="R180" xref="yes"/>
+<wire x1="233.68" y1="53.34" x2="228.6" y2="53.34" width="0.1524" layer="91"/>
 </segment>
 </net>
@@
 <segment>
 <pinref part="JP1" gate="A" pin="2"/>
-<wire x1="238.76" y1="66.04" x2="226.06" y2="66.04" width="0.1524" layer="91"/>
-<label x="226.06" y="66.04" size="1.778" layer="95" rot="R180" xref="yes"/>
+<wire x1="233.68" y1="55.88" x2="220.98" y2="55.88" width="0.1524" layer="91"/>
+<label x="220.98" y="55.88" size="1.778" layer="95" rot="R180" xref="yes"/>
 </segment>
 </net>
@@
 <pinref part="JP1" gate="A" pin="6"/>
 <pinref part="GND1" gate="1" pin="GND"/>
-<wire x1="223.52" y1="55.88" x2="238.76" y2="55.88" width="0.1524" layer="91"/>
+<wire x1="218.44" y1="45.72" x2="233.68" y2="45.72" width="0.1524" layer="91"/>
 </segment>
 <segment>
 <pinref part="S1" gate="G$1" pin="2"/>
 <pinref part="GND6" gate="1" pin="GND"/>
-<wire x1="60.96" y1="60.96" x2="63.5" y2="60.96" width="0.1524" layer="91"/>
+<wire x1="144.78" y1="48.26" x2="147.32" y2="48.26" width="0.1524" layer="91"/>
 </segment>
 <segment>
 <pinref part="S2" gate="G$1" pin="2"/>
 <pinref part="GND5" gate="1" pin="GND"/>
-<wire x1="60.96" y1="35.56" x2="63.5" y2="35.56" width="0.1524" layer="91"/>
+<wire x1="58.42" y1="48.26" x2="60.96" y2="48.26" width="0.1524" layer="91"/>
 </segment>
 <segment>
@@
 <pinref part="+3V3" gate="G$1" pin="+3V3"/>
 <pinref part="R1" gate="G$1" pin="1"/>
-<wire x1="35.56" y1="60.96" x2="38.1" y2="60.96" width="0.1524" layer="91"/>
+<wire x1="119.38" y1="48.26" x2="121.92" y2="48.26" width="0.1524" layer="91"/>
 </segment>
 <segment>
 <pinref part="+3V4" gate="G$1" pin="+3V3"/>
 <pinref part="R2" gate="G$1" pin="1"/>
-<wire x1="35.56" y1="35.56" x2="38.1" y2="35.56" width="0.1524" layer="91"/>
+<wire x1="33.02" y1="48.26" x2="35.56" y2="48.26" width="0.1524" layer="91"/>
 </segment>
 <segment>
@@
 <pinref part="+3V5" gate="G$1" pin="+3V3"/>
 <pinref part="SJ1" gate="1" pin="1"/>
-<wire x1="213.36" y1="60.96" x2="215.9" y2="60.96" width="0.1524" layer="91"/>
+<wire x1="208.28" y1="50.8" x2="210.82" y2="50.8" width="0.1524" layer="91"/>
 </segment>
 <segment>
@@
 <pinref part="SJ1" gate="1" pin="2"/>
 <pinref part="JP1" gate="A" pin="4"/>
-<wire x1="226.06" y1="60.96" x2="238.76" y2="60.96" width="0.1524" layer="91"/>
-</segment>
-</net>
+<wire x1="220.98" y1="50.8" x2="233.68" y2="50.8" width="0.1524" layer="91"/>
+</segment>
+</net>
